Commit message: UPDATE: base_controller.cpp and base_controller.py. Both Nodes should do the same now

File: src/robot_urdf/urdf/robot.urdf (robot description, URDF)
Before this commit: robot myRobot, 5 links, 4 joints
Links:
- link base_link: geometry visual box size=0.360 0.290 0.070

Commit message: UPDATE: robot.urdf; ADD: new launchfile for package robot_urdf, robot_rviz.launch

File: src/robot_urdf/urdf/robot.urdf (robot description, URDF)
Before this commit: robot myRobot, 5 links, 4 joints
Joints:
- joint base_to_l_front_wheel: axis (none) -> 0 1 0; origin xyz=0 0 0 -> xyz=-.1475 .1775 .035 rpy=0 0 0; type fixed -> continuous
- joint base_to_l_rear_wheel: axis (none) -> 0 1 0; origin xyz=0 0 0 -> xyz=-.1475 -.1775 .035 rpy=0 0 0; type fixed -> continuous
- joint base_to_r_front_wheel: axis (none) -> 0 1 0; origin xyz=0 0 0 -> xyz=.1475 .1775 .035 rpy=0 0 0; type fixed -> continuous
- joint base_to_r_rear_wheel: axis (none) -> 0 1 0; origin xyz=0 0 0 -> xyz=.1475 -.1775 .035 rpy=0 0 0; type fixed -> continuous

Commit message: UPDATE serialport_defaults.yaml. UPDATE base_odometry_node cpp, now transform send from odom to base_footprint. UPDATE robot.urdf, implemented link base_footprint as parent of base_link

File: src/robot_urdf/urdf/robot.urdf (robot description, URDF)
Before this commit: robot robot, 5 links, 4 joints
Links:
- added link base_footprint
Joints:
- added joint base_footprint_to_base_link: type fixed, parent base_footprint, child base_link, origin xyz=0 0 0.035 rpy=0 0 0

Commit message: UPDATE: robot.urdf

File: src/robot_urdf/urdf/robot.urdf (robot description, URDF)
Before this commit: robot robot, 6 links, 5 joints
Joints:
- joint base_to_l_front_wheel: origin xyz=-.1475 .1775 .035 rpy=0 0 0 -> xyz=-.1475 .1775 0 rpy=0 0 0
- joint base_to_l_rear_wheel: origin xyz=-.1475 -.1775 .035 rpy=0 0 0 -> xyz=-.1475 -.1775 0 rpy=0 0 0
- joint base_to_r_front_wheel: origin xyz=.1475 .1775 .035 rpy=0 0 0 -> xyz=.1475 .1775 0 rpy=0 0 0
- joint base_to_r_rear_wheel: origin xyz=.1475 -.1775 .035 rpy=0 0 0 -> xyz=.1475 -.1775 0 rpy=0 0 0

Commit message: UPDATE format of some yaml-Files. UPDATE robot.urdf

File: src/robot_urdf/urdf/robot.urdf (robot description, URDF)
Before this commit: robot robot, 6 links, 5 joints
Links:
- link base_link: geometry collision box size=0.360 0.290 0.070; visual box size=0.360 0.290 0.070
- link l_front_wheel: geometry collision cylinder length=0.065 radius=0.035; visual cylinder length=0.065 radius=0.035
- link l_rear_wheel: geometry collision cylinder length=0.065 radius=0.035; visual cylinder length=0.065 radius=0.035
- link r_front_wheel: geometry collision cylinder length=0.065 radius=0.035; visual cylinder length=0.065 radius=0.035
- link r_rear_wheel: geometry collision cylinder length=0.065 radius=0.035; visual cylinder length=0.065 radius=0.035
Joints:
- removed joint base_footprint_to_base_link
- removed joint base_to_l_front_wheel
- removed joint base_to_l_rear_wheel
- removed joint base_to_r_front_wheel
- removed joint base_to_r_rear_wheel
- added joint base_footprint_joint: type fixed, parent base_footprint, child base_link, origin xyz=0 0 0.035 rpy=0 0 0
- added joint l_front_wheel_joint: type continuous, parent base_link, child l_front_wheel, origin xyz=.1475 .1775 0 rpy=0 0 0, axis 0 1 0
- added joint l_rear_wheel_joint: type continuous, parent base_link, child l_rear_wheel, origin xyz=-.1475 .1775 0 rpy=0 0 0, axis 0 1 0
- added joint r_front_wheel_joint: type continuous, parent base_link, child r_front_wheel, origin xyz=.1475 -.1775 0 rpy=0 0 0, axis 0 1 0
- added joint r_rear_wheel_joint: type continuous, parent base_link, child r_rear_wheel, origin xyz=-.1475 -.1775 0 rpy=0 0 0, axis 0 1 0

Commit message: UPDATE robot.urdf

File: src/robot_urdf/urdf/robot.urdf (robot description, URDF)
Before this commit: robot robot, 6 links, 5 joints
Links:
- added link l_track; collision box size=0.290 0.065 0.070; visual box size=0.290 0.065 0.070
- added link r_track; collision box size=0.290 0.065 0.070; visual box size=0.290 0.065 0.070
Joints:
- added joint l_track_joint: type fixed, parent base_link, child l_track, origin xyz=0 0.1775 0 rpy=0 0 0
- added joint r_track_joint: type fixed, parent base_link, child r_track, origin xyz=0 -0.1775 0 rpy=0 0 0

Commit message: UPDATE robot.urdf: connect wheels via joint mimic tag

File: src/robot_urdf/urdf/robot.urdf (robot description, URDF)
Before this commit: robot robot, 8 links, 7 joints
Joints:
- joint l_front_wheel_joint: mimic (none) -> joint=l_rear_wheel_joint offset=0.0
- joint r_front_wheel_joint: mimic (none) -> joint=r_rear_wheel_joint offset=0.0

Commit message: UPDATE robot.urdf: Added torso and kinect

File: src/robot_urdf/urdf/robot.urdf (robot description, URDF)
Before this commit: robot robot, 8 links, 7 joints
Links:
- added link camera_depth_frame, mass 0.0001
- added link kinect_depth_optical_frame, mass 0.0001
- added link kinect_link, mass 0.0001; visual box size=0.064 0.280 0.03
- added link torso; collision box size=0.360 0.290 0.070; visual box size=0.360 0.420 0.120
Joints:
- added joint depth_optical_joint: type fixed, parent camera_depth_frame, child kinect_depth_optical_frame, origin xyz=0 0 0 rpy=1.57075 0 -1.57075
- added joint kinect_depth_joint: type fixed, parent kinect_link, child camera_depth_frame, origin xyz=0 0.028 0 rpy=0 0 0
- added joint kinect_link_to_torso: type fixed, parent torso, child kinect_link, origin xyz=0.148 0 0.075 rpy=0 0 0
- added joint torso_joint: type fixed, parent base_link, child torso, origin xyz=0 0 0.098 rpy=0 0 0
- joint l_front_wheel_joint: origin xyz=.1475 .1775 0 rpy=0 0 0 -> xyz=.1475 .1775 0 rpy=1.57075 0 0
- joint l_rear_wheel_joint: origin xyz=-.1475 .1775 0 rpy=0 0 0 -> xyz=-.1475 .1775 0 rpy=1.57075 0 0
- joint r_front_wheel_joint: origin xyz=.1475 -.1775 0 rpy=0 0 0 -> xyz=.1475 -.1775 0 rpy=1.57075 0 0
- joint r_rear_wheel_joint: origin xyz=-.1475 -.1775 0 rpy=0 0 0 -> xyz=-.1475 -.1775 0 rpy=1.57075 0 0

Commit message: UPDATE robot.urdf: Changed some frame names and color of torso and baase_link

File: src/robot_urdf/urdf/robot.urdf (robot description, URDF)
Before this commit: robot robot, 12 links, 11 joints
Links:
- removed link kinect_link
- added link camera_link, mass 0.0001; visual box size=0.064 0.280 0.03
Joints:
- removed joint kinect_link_to_torso
- added joint camera_link_to_torso: type fixed, parent torso, child camera_link, origin xyz=0.148 0 0.075 rpy=0 0 0
- joint kinect_depth_joint: parent kinect_link -> camera_link

Commit message: UPDATE robot.urdf: Kinect is no rendered from a mesh file

File: src/robot_urdf/urdf/robot.urdf (robot description, URDF)
Before this commit: robot robot, 12 links, 11 joints
Links:
- removed link kinect_depth_optical_frame
- added link camera_depth_optical_frame, mass 0.001
- added link camera_rgb_frame, mass 0.001
- added link camera_rgb_optical_frame, mass 0.001
- link camera_depth_frame: mass 0.0001 -> 0.001
- link camera_link: mass 0.0001 -> 0.001; geometry collision box size=0.07271 0.27794 0.073; visual mesh filename=package://robot_urdf/meshes/sensors/kinect.dae
Joints:
- removed joint camera_link_to_torso
- removed joint depth_optical_joint
- removed joint kinect_depth_joint
- added joint camera_depth_joint: type fixed, parent camera_rgb_frame, child camera_depth_frame, origin xyz=0 0.0250 0 rpy=0 0 0
- added joint camera_depth_optical_joint: type fixed, parent camera_depth_frame, child camera_depth_optical_frame, origin xyz=0 0 0 rpy=-1.5707 0 -1.5707
- added joint camera_joint: type fixed, parent camera_rgb_frame, child camera_link, origin xyz=-0.031 -0.0125 -0.016 rpy=0 0 0
- added joint camera_rgb_joint: type fixed, parent torso, child camera_rgb_frame, origin xyz=0.148 0 0.0965 rpy=0 0 0
- added joint camera_rgb_optical_joint: type fixed, parent camera_rgb_frame, child camera_rgb_optical_frame, origin xyz=0 0 0 rpy=-1.5707 0 -1.5707

Commit message: UPDATE robot.urdf: Switched back to simpler urdf description for kinect, but kept mesh file for kinect

File: src/robot_urdf/urdf/robot.urdf (robot description, URDF)
Before this commit: robot robot, 14 links, 13 joints
Links:
- removed link camera_depth_optical_frame
- removed link camera_rgb_frame
- removed link camera_rgb_optical_frame
- added link kinect_depth_optical_frame, mass 0.0001
- link camera_depth_frame: mass 0.001 -> 0.0001
Joints:
- removed joint camera_depth_joint
- removed joint camera_depth_optical_joint
- removed joint camera_joint
- removed joint camera_rgb_joint
- removed joint camera_rgb_optical_joint
- added joint camera_link_to_torso: type fixed, parent torso, child camera_link, origin xyz=0.148 0 0.0965 rpy=0 0 0
- added joint depth_optical_joint: type fixed, parent camera_depth_frame, child kinect_depth_optical_frame, origin xyz=0 0 0 rpy=1.57075 0 -1.57075
- added joint kinect_depth_joint: type fixed, parent camera_link, child camera_depth_frame, origin xyz=0 0.028 0 rpy=0 0 0
